File: board/SPv0/SPv0.brd (EAGLE design)
At the start: 97 x 24.6 mm, 39 parts, among them IC1 S34ML0XG1, IC2 F55[0/1]X---PT48, IC4 74LS14D, Q1 12MHz

Commit message: halfboard v1 done!
Parts:
- added SJ1: (no value), jumper:SJW
- moved R7 47.2 mm to (27.4, 30.9)
- moved R6 43.4 mm to (27.4, 29.0), turned to 180 degrees
- moved IC4 41.0 mm to (34.3, 29.5), turned to 180 degrees
- moved U$1 15.8 mm to (46.5, 29.2), turned to 180 degrees
- moved R5 12.0 mm to (27.5, 33.0), turned to 180 degrees
- moved R4 11.2 mm to (21.6, 27.9), turned to 225 degrees
- moved C6 6.55 mm to (16.8, 32.1), turned to 225 degrees
- moved TP4 4.83 mm to (16.4, 18.8), flipped to the top
- moved C7 3.46 mm to (13.4, 28.9), turned to 45 degrees
- moved TP1 3.42 mm to (16.5, 20.7), flipped to the top
- moved Q1 1.59 mm to (17.3, 28.1), turned to 225 degrees
- moved C3 1.42 mm to (23.2, 26.7), turned to 225 degrees
- moved TP3 1.05 mm to (27.7, 8.13), flipped to the top
- moved TP5 1.00 mm to (15.2, 17.0), flipped to the top
- turned C2 to 90 degrees
Connections:
- new net N$11: R4.P$2, SJ1.1
- new net SW_A: IC2.4, U$1.P$2
- net GND: now also U$1.P$1
- net N$4: now also SJ1.2; no longer U$1.P$2
- net PUR_A: no longer R4.P$2, U$1.P$1
Routing:
- net GND: track 0.00 -> 171.2 mm, vias 0 -> 13
- net +3V3_A: track 6.86 -> 98.1 mm, vias 0 -> 2
- net VCC: track 49.1 -> 102.0 mm, vias 2 -> 0
- net VBUS: track 3.37 -> 46.1 mm, vias 0 -> 2
- net SW_A: track 0.00 -> 31.0 mm, vias 0 -> 2
- net D+_A: track 0.00 -> 20.5 mm, vias 0 -> 2
- net DOUT: track 0.00 -> 19.4 mm, vias 0 -> 2
- net D-_A: track 0.00 -> 17.1 mm, vias 0 -> 2
- net !RST_A!: track 0.00 -> 16.3 mm, vias 0 -> 2
- net XT2IN_A: track 0.00 -> 15.5 mm
- net N$7: track 0.00 -> 12.7 mm, vias 0 -> 2
- net XT2OUT_A: track 0.00 -> 11.0 mm
- net N$9: track 0.00 -> 8.47 mm
- net +1V8_A: track 0.00 -> 8.23 mm, vias 0 -> 2
- net N$10: track 0.00 -> 5.61 mm
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- removed copper zone on layer 16, net GND
Other:
- board size 97 x 24.6 mm -> 56.4 x 27.9 mm
