File: board/SPv2/SPv2.2.brd (EAGLE design)
At the start: 56.5 x 22.9 mm, 38 parts, among them IC1 S34ML0XG1, IC2 F5508, IC4 74LS14DB, Q1 12MHz

Commit message: finalizing half-board, switch testing remains
Parts:
- removed U$1: KMR-2, Passives:KMR-2-SWITCH
- added SW1: KMR-2, Passives:KMR-2-SWITCH
- moved U$2 0.35 mm to (58.7, 11.4)
Connections:
- net GND: now also SW1.PA1, SW1.PA2; no longer U$1.PA1, U$1.PA2
- net SW_A: now also SW1.PB1, SW1.PB2; no longer U$1.PB1, U$1.PB2
Routing:
- net SW_A: track 36.6 -> 42.5 mm
- net GND: track 163.6 -> 167.4 mm
- net VBUS: track 88.8 -> 89.8 mm
Other:
- board size 56.5 x 22.9 mm -> 56.2 x 22.9 mm
- board text added: "(c)2014-5 phooky"
- board text added: "v0.2.3"
